File: kicad/donttouchit/donttouchit.kicad_pcb (KiCad board)
At the start: 2 copper layers, 45 x 51.5 mm, 33 parts, among them J1 Conn_01x02_Female, J10 Conn_01x04_Male, J2 Conn_01x02_Female, J3 Conn_01x02_Female, J7 Conn_01x02_Female, J8 Conn_01x02_Female, J9 Conn_01x02_Female, U1 LDC1614, U2 TMP112xxDRL

Commit message: V1.2 fabrication files generated
Parts:
- C10, C4, C5, C6, C7, C8: value 100n -> 12p
- U2: value TMP112xxDRL -> TMP112NAIDRLR
Changed lines of the file:
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@@
     (fp_line (start 2 2) (end -2 2)
       (stroke (width 0.1) (type solid)) (layer "F.Fab"))
-    (pad "" smd roundrect (at -0.65 -0.65) (size 1.13 1.13) (layers "F.Paste") (roundrect_rratio 0.221239))
-    (pad "" smd roundrect (at -0.65 0.65) (size 1.13 1.13) (layers "F.Paste") (roundrect_rratio 0.221239))
-    (pad "" smd roundrect (at 0.65 -0.65) (size 1.13 1.13) (layers "F.Paste") (roundrect_rratio 0.221239))
-    (pad "" smd roundrect (at 0.65 0.65) (size 1.13 1.13) (layers "F.Paste") (roundrect_rratio 0.221239))
+    (pad "" smd roundrect (at -0.65 -0.65) (size 1.13 1.13) (layers "F.Paste") (roundrect_rratio 0.2212389381))
+    (pad "" smd roundrect (at -0.65 0.65) (size 1.13 1.13) (layers "F.Paste") (roundrect_rratio 0.2212389381))
+    (pad "" smd roundrect (at 0.65 -0.65) (size 1.13 1.13) (layers "F.Paste") (roundrect_rratio 0.2212389381))
+    (pad "" smd roundrect (at 0.65 0.65) (size 1.13 1.13) (layers "F.Paste") (roundrect_rratio 0.2212389381))
     (pad "1" smd roundrect (at -1.9375 -0.75) (size 0.875 0.25) (layers "F.Cu" "F.Paste" "F.Mask") (roundrect_rratio 0.25)
       (net 10 "Net-(J10-Pin_3)") (pinfunction "SCL") (pintype "input"))
@@
         (effects (font (size 0.8 0.8) (thickness 0.15)))
     )
-    (fp_text value "100n" (at 0 1.43) (layer "F.Fab")
+    (fp_text value "12p" (at 0 1.43) (layer "F.Fab")
         (effects (font (size 1 1) (thickness 0.15)))
     )
@@
         (effects (font (size 0.8 0.8) (thickness 0.15)))
     )
-    (fp_text value "100n" (at 0 1.43 -270) (layer "F.Fab")
+    (fp_text value "12p" (at 0 1.43 -270) (layer "F.Fab")
         (effects (font (size 1 1) (thickness 0.15)))
     )
@@
         (effects (font (size 0.8 0.8) (thickness 0.15)))
     )
-    (fp_text value "100n" (at 0 1.43) (layer "F.Fab")
+    (fp_text value "12p" (at 0 1.43) (layer "F.Fab")
         (effects (font (size 1 1) (thickness 0.15)))
     )
@@
         (effects (font (size 0.8 0.8) (thickness 0.15)))
     )
-    (fp_text value "100n" (at 0 1.43) (layer "F.Fab")
+    (fp_text value "12p" (at 0 1.43) (layer "F.Fab")
         (effects (font (size 1 1) (thickness 0.15)))
     )
@@
         (effects (font (size 0.8 0.8) (thickness 0.15)))
     )
-    (fp_text value "TMP112xxDRL" (at 0 1.75) (layer "F.Fab")
+    (fp_text value "TMP112NAIDRLR" (at 0 1.75) (layer "F.Fab")
         (effects (font (size 1 1) (thickness 0.15)))
     )
@@
         (effects (font (size 0.8 0.8) (thickness 0.15)))
     )
-    (fp_text value "100n" (at 0 1.43) (layer "F.Fab")
+    (fp_text value "12p" (at 0 1.43) (layer "F.Fab")
         (effects (font (size 1 1) (thickness 0.15)))
     )
@@
         (effects (font (size 0.8 0.8) (thickness 0.15)))
     )
-    (fp_text value "100n" (at 0 1.43 90) (layer "F.Fab")
-        (effects (font (size 1 1) (thickness 0.15)))
-    )
+    (fp_text value "12p" (at 0 1.43 90) (layer "F.Fab")
+        (effects (font (size 1 1) (thickness 0.15)))
+    )
